File: pcb/esp-butt/esp-butt.kicad_sch (KiCad schematic)
At the start: 20 parts, among them J1 1x04_P2.54mm, J2 JST_XH_B2B, U1 XIAO-ESP32-C3

Commit message: More stuffs
Parts:
- J2: value JST_XH_B2B -> JST_PH; footprint Connector_JST:JST_XH_B2B-XH-A_1x02_P2.50mm_Vertical -> Connector_JST:JST_PH_B2B-PH-K_1x02_P2.00mm_Vertical
Changed lines of the file:
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@@
 			)
 		)
-		(property "Value" "JST_XH_B2B"
-			(at 101.6 45.72 0)
+		(property "Value" "JST_PH"
+			(at 104.14 45.72 0)
 			(effects
 				(font
@@
 			)
 		)
-		(property "Footprint" "Connector_JST:JST_XH_B2B-XH-A_1x02_P2.50mm_Vertical"
+		(property "Footprint" "Connector_JST:JST_PH_B2B-PH-K_1x02_P2.00mm_Vertical"
 			(at 109.22 40.64 0)
 			(effects

Commit message: workies
Parts:
- removed H1, H2: MountingHole, MountingHole:MountingHole_2.2mm_M2, symbol Mechanical:MountingHole

Commit message: More work + docs
Parts:
- added BATT1: 3.7V LiPo 600mAH, symbol esp-butt:Battery
- added D1: 1.3 inch OLED I2C 128 x 64, symbol esp-butt:OLED_128x64_1.3in_I2C
- C1, C2: Source_US (none) -> https://www.digikey.dk/short/hbr1hz4m; Value_ALT (none) -> 0,1μF
- C3: Source_US (none) -> https://www.digikey.dk/short/v7fv0pbn; Value_ALT (none) -> 10000pF
- J1: Source_US (none) -> https://www.digikey.dk/short/pz373nw5
- R7, R8: Source_US (none) -> https://www.digikey.dk/short/2qbtnbbv
- S1: Source_US (none) -> https://www.digikey.dk/short/bdcwrr3h
- S2: Source_US (none) -> https://www.digikey.dk/short/0qr8pj0r
- U1: Source_US (none) -> https://www.digikey.dk/short/rv35rpwt
Other:
- moved on the sheet: J1

Commit message: Add Pillow dependency and implement session recording feature
- Added "pillow" to dependencies in pyproject.toml and uv.lock.
- Enhanced HardwareMock to support session recording, including:
  - New spawn_recorder_task function to handle event and frame recording.
  - Logic to create a temporary directory for storing frames.
  - Recording navigation and slider events to a specified NDJSON file.
  - Saving frames as PNG images during the session.
Parts:
- C1, C2: Value_ALT 0,1μF -> (none)
- C3: Value_ALT 10000pF -> (none)
Changed lines of the file:
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@@
 			)
 		)
-		(property "Value_ALT" ""
-			(at 104.14 80.01 0)
-			(hide yes)
-			(show_name no)
-			(do_not_autoplace no)
-			(effects
-				(font
-					(size 1.27 1.27)
-				)
-			)
-		)
 		(instances
 			(project "esp-butt"
@@
 			)
 		)
-		(property "Value_ALT" ""
-			(at 26.67 109.22 90)
-			(hide yes)
-			(show_name no)
-			(do_not_autoplace no)
-			(effects
-				(font
-					(size 1.27 1.27)
-				)
-			)
-		)
 		(pin "2"
 		)
@@
 			)
 		)
-		(property "Value_ALT" ""
-			(at 99.06 29.21 90)
-			(hide yes)
-			(show_name no)
-			(do_not_autoplace no)
-			(effects
-				(font
-					(size 1.27 1.27)
-				)
-			)
-		)
 		(pin "2"
 		)
@@
 			)
 		)
-		(property "Value_ALT" ""
-			(at 142.24 35.56 0)
-			(hide yes)
-			(show_name no)
-			(do_not_autoplace no)
-			(effects
-				(font
-					(size 1.27 1.27)
-				)
-			)
-		)
 		(pin "2"
 		)
@@
 			)
 		)
-		(property "Value_ALT" ""
-			(at 146.05 88.9 0)
-			(hide yes)
-			(show_name no)
-			(do_not_autoplace no)
-			(effects
-				(font
-					(size 1.27 1.27)
-				)
-			)
-		)
 		(pin "2"
 		)
@@
 			)
 		)
-		(property "Value_ALT" ""
-			(at 99.06 39.37 90)
-			(hide yes)
-			(show_name no)
-			(do_not_autoplace no)
-			(effects
-				(font
-					(size 1.27 1.27)
-				)
-			)
-		)
 		(pin "2"
 		)
@@
 			)
 		)
-		(property "Value_ALT" ""
-			(at 109.22 40.64 0)
-			(hide yes)
-			(show_name no)
-			(do_not_autoplace no)
-			(effects
-				(font
-					(size 1.27 1.27)
-				)
-			)
-		)
 		(pin "2"
 		)
@@
 			)
 		)
-		(property "Value_ALT" ""
-			(at 41.91 49.53 0)
-			(hide yes)
-			(show_name no)
-			(do_not_autoplace no)
-			(effects
-				(font
-					(size 1.27 1.27)
-				)
-			)
-		)
 		(pin "14"
 		)
@@
 			)
 		)
-		(property "Value_ALT" "0,1μF"
-			(at 21.59 113.03 0)
-			(hide yes)
-			(show_name no)
-			(do_not_autoplace no)
-			(effects
-				(font
-					(size 1.27 1.27)
-				)
-			)
-		)
 		(pin "1"
 		)
@@
 			)
 		)
-		(property "Value_ALT" ""
-			(at 102.87 16.51 0)
-			(hide yes)
-			(show_name no)
-			(do_not_autoplace no)
-			(effects
-				(font
-					(size 1.27 1.27)
-				)
-			)
-		)
 		(instances
 			(project "esp-butt"
@@
 			)
 		)
-		(property "Value_ALT" ""
-			(at 106.68 113.03 90)
-			(hide yes)
-			(show_name no)
-			(do_not_autoplace no)
-			(effects
-				(font
-					(size 1.27 1.27)
-				)
-			)
-		)
 		(pin "1"
 		)
@@
 			)
 		)
-		(property "Value_ALT" ""
-			(at 109.22 67.31 0)
-			(hide yes)
-			(show_name no)
-			(do_not_autoplace no)
-			(effects
-				(font
-					(size 1.27 1.27)
-				)
-			)
-		)
 		(pin "4"
 		)
@@
 			)
 		)
-		(property "Value_ALT" "10000pF"
-			(at 113.03 118.11 0)
-			(hide yes)
-			(show_name no)
-			(do_not_autoplace no)
-			(effects
-				(font
-					(size 1.27 1.27)
-				)
-			)
-		)
 		(pin "2"
 		)
@@
 			)
 		)
-		(property "Value_ALT" ""
-			(at 31.75 104.14 90)
-			(hide yes)
-			(show_name no)
-			(do_not_autoplace no)
-			(effects
-				(font
-					(size 1.27 1.27)
-				)
-			)
-		)
 		(pin "2"
 		)
@@
 			)
 		)
-		(property "Value_ALT" "0,1μF"
-			(at 46.99 113.03 0)
-			(hide yes)
-			(show_name no)
-			(do_not_autoplace no)
-			(effects
-				(font
-					(size 1.27 1.27)
-				)
-			)
-		)
 		(pin "1"
 		)
@@
 			)
 		)
-		(property "Value_ALT" ""
-			(at 146.05 68.58 0)
-			(hide yes)
-			(show_name no)
-			(do_not_autoplace no)
-			(effects
-				(font
-					(size 1.27 1.27)
-				)
-			)
-		)
 		(pin "2"
 		)
@@
 			)
 		)
-		(property "Value_ALT" ""
-			(at 41.91 109.22 90)
-			(hide yes)
-			(show_name no)
-			(do_not_autoplace no)
-			(effects
-				(font
-					(size 1.27 1.27)
-				)
-			)
-		)
 		(pin "2"
 		)
@@
 			)
 		)
-		(property "Value_ALT" ""
-			(at 113.03 106.68 90)
-			(hide yes)
-			(show_name no)
-			(do_not_autoplace no)
-			(effects
-				(font
-					(size 1.27 1.27)
-				)
-			)
-		)
 		(pin "1"
 		)
@@
 			)
 		)
-		(property "Value_ALT" ""
-			(at 87.63 109.22 0)
-			(hide yes)
-			(show_name no)
-			(do_not_autoplace no)
-			(effects
-				(font
-					(size 1.27 1.27)
-				)
-			)
-		)
 		(pin "1"
 		)
@@
 			(at 36.83 104.14 90)
 			(hide yes)
-			(show_name no)
-			(do_not_autoplace no)
-			(effects
-				(font
-					(size 1.27 1.27)
-				)
-			)
-		)
-		(property "Value_ALT" ""
-			(at 36.83 104.14 90)
-			(hide yes)

Commit message: Documentation updates
Parts:
- C1, C2: Value_ALT (none) -> 10000pF
- C3: Value_ALT (none) -> 0.1uF
- J1: value 1x04_P2.54mm -> 1x04 2.54mm
- J2: value JST_PH -> 1x02 JST_PH; Value_ALT (none) -> B2B (vertical)
- R7, R8: footprint esp-butt:TRIM_PTA4543-2015DPB103 -> PTA4543-2015DPB103:TRIM_PTA4543-2015DPB103; MFN PTA4543-2015DPB103-ND -> (none); Source_US https://www.digikey.dk/short/2qbtnbbv -> (none); Value_ALT (none) -> 10k±20%, 0.25W Linear
- U1: value XIAO-ESP32-C3 -> XIAO-ESP32-S3
